Commit message: Improve crack fidelity and state-driven repair simulation

File: src/repairman_vision/urdf/repairman_demo.urdf (robot description, URDF)
Before this commit: robot repairman_demo, 4 links, 3 joints
Links:
- removed link mast_link
- added link link_1; visual cylinder length=0.06 radius=0.08
- added link link_2; visual cylinder length=0.28 radius=0.045; visual sphere radius=0.055
- added link link_3; visual cylinder length=0.24 radius=0.040; visual sphere radius=0.048
- added link link_4; visual cylinder length=0.09 radius=0.032
- added link link_5; visual cylinder length=0.09 radius=0.028
- added link link_6; visual cylinder length=0.10 radius=0.024
- added link tool_flange; visual cylinder length=0.03 radius=0.022
- link base_link: geometry visual cylinder length=0.04 radius=0.12; visual cylinder length=0.11 radius=0.17
- link tool_link: geometry visual cylinder length=0.10 radius=0.010; visual sphere radius=0.012
Joints:
- removed joint base_to_mast
- removed joint mast_to_tool
- added joint joint_1: type revolute, parent base_link, child link_1, origin xyz=0 0 0.14 rpy=0 0 0, axis 0 0 1, limit lower=-3.14159 upper=3.14159 effort=250 velocity=2.5
- added joint joint_2: type revolute, parent link_1, child link_2, origin xyz=0 0 0.03 rpy=0 0 0, axis 0 1 0, limit lower=-2.60 upper=2.60 effort=220 velocity=2.2
- added joint joint_3: type revolute, parent link_2, child link_3, origin xyz=0.28 0 0 rpy=0 0 0, axis 0 1 0, limit lower=-2.80 upper=2.80 effort=180 velocity=2.2
- added joint joint_4: type revolute, parent link_3, child link_4, origin xyz=0.24 0 0 rpy=0 0 0, axis 0 0 1, limit lower=-3.14159 upper=3.14159 effort=140 velocity=3.1
- added joint joint_5: type revolute, parent link_4, child link_5, origin xyz=0.09 0 0 rpy=0 0 0, axis 0 1 0, limit lower=-2.60 upper=2.60 effort=120 velocity=3.1
- added joint joint_6: type revolute, parent link_5, child link_6, origin xyz=0.09 0 0 rpy=0 0 0, axis 0 0 1, limit lower=-6.28318 upper=6.28318 effort=90 velocity=3.8
- added joint tool_fixed: type fixed, parent tool_flange, child tool_link, origin xyz=0.03 0 0 rpy=0 0 0
- added joint tool_flange_joint: type fixed, parent link_6, child tool_flange, origin xyz=0.10 0 0 rpy=0 0 0
